File: tests/corpus/goldens/design.kicad_sch (KiCad schematic)
At the start: 1 part, among them J1 Header_2x1

Commit message: fix(kicad): portable verified libraries; retain J1/D1 ERC blockers (#116)
* fix(kicad): export portable verified symbol and footprint libraries

* test(kicad): refresh qualified symbol-ID golden fixture

* fix(kicad): bound portable library paths and align export tests

* security(kicad): normalize and bound portable export paths

* security(kicad): resolve library members without writing workspace root

* test(kicad): refresh portable symbol artifact integrity snapshots
Parts:
- J1: symbol ZapTrace_J1 -> ZapTrace:ZapTrace_J1
Changed lines of the file:
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@@
   )
   (symbol
-    (lib_id "ZapTrace_R1")
+    (lib_id "ZapTrace:ZapTrace_R1")
     (at 50.8 50.8 0)
     (unit 1)
@@
   )
   (symbol
-    (lib_id "ZapTrace_R2")
+    (lib_id "ZapTrace:ZapTrace_R2")
     (at 101.6 50.8 0)
     (unit 1)
@@
   )
   (symbol
-    (lib_id "ZapTrace_C1")
+    (lib_id "ZapTrace:ZapTrace_C1")
     (at 152.4 50.8 0)
     (unit 1)
@@
   )
   (symbol
-    (lib_id "ZapTrace_J1")
+    (lib_id "ZapTrace:ZapTrace_J1")
     (at 203.2 50.8 0)
     (unit 1)
